File: Channel2Photodetect.sch (KiCad schematic (older format))
At the start: 7 parts, among them U201 MCP6404, U202 LM339

Commit message: revised feedback resistor and updated reference voltage divider
Parts:
- removed R302: 22M, Resistors_SMD:R_0805_HandSoldering, symbol R_Small
- C301: value 2.2p -> 50p
- R301: value 22M -> 2M; Fieldname (none) -> Value; MPN RMCF0805FT22M0 -> (none)
- renumbered R303 to R302
Connections:
- net at C301.1, R302.2, U201.7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: now also R301.1
Changed lines of the file:
@@
 P 5210 2100
 F 0 "C301" V 5330 2060 50  0000 L CNN
-F 1 "2.2p" V 5100 1970 50  0000 L CNN
+F 1 "50p" V 5100 1970 50  0000 L CNN
 F 2 "Capacitors_SMD:C_0805_HandSoldering" H 5210 2100 50  0001 C CNN
 F 3 "" H 5210 2100 50  0000 C CNN
@@
 	4800 3250 4800 3550
 $Comp
-L R_Small R303
+L R_Small R302
 U 1 1 5822914A
 P 5610 3550
-F 0 "R303" V 5690 3510 50  0000 L CNN
+F 0 "R302" V 5690 3510 50  0000 L CNN
 F 1 "10K" V 5540 3430 50  0000 L CNN
 F 2 "Resistors_SMD:R_0805_HandSoldering" H 5610 3550 50  0001 C CNN
@@
 P 4980 2620
 F 0 "R301" V 5060 2580 50  0000 L CNN
-F 1 "22M" V 4910 2500 50  0000 L CNN
+F 1 "2M" V 4910 2500 50  0000 L CNN
 F 2 "Resistors_SMD:R_0805_HandSoldering" H 4980 2620 50  0001 C CNN
 F 3 "" H 4980 2620 50  0000 C CNN
-F 4 "RMCF0805FT22M0" H 4980 2620 60  0001 C CNN "MPN"
+F 4 "Value" H 4980 2620 60  0001 C CNN "Fieldname"
 	1    4980 2620
 	0    1    1    0
 $EndComp
-$Comp
-L R_Small R302
-U 1 1 5823C7D9
-P 5310 2620
-F 0 "R302" V 5390 2580 50  0000 L CNN
-F 1 "22M" V 5240 2500 50  0000 L CNN
-F 2 "Resistors_SMD:R_0805_HandSoldering" H 5310 2620 50  0001 C CNN
-F 3 "" H 5310 2620 50  0000 C CNN
-F 4 "RMCF0805FT22M0" H 5310 2620 60  0001 C CNN "MPN"
-	1    5310 2620
-	0    1    1    0
-$EndComp
 Wire Wire Line
-	5410 2620 5610 2620
-Wire Wire Line
-	5210 2620 5080 2620
+	5610 2620 5080 2620
 Wire Wire Line
 	4880 2620 4800 2620

Commit message: added pull-up resistors
Parts:
- added R303: 10K, Resistors_SMD:R_0805_HandSoldering, symbol R_Small
- R301: Fieldname Value -> (none); MPN (none) -> RC0805FR-072ML
- U202: MPN (none) -> LM339DE4
Connections:
- net PD2: now also R303.1
- new net +3V: R303.2
Changed lines of the file:
@@
 F 2 "Housings_SOIC:SOIC-14_3.9x8.7mm_Pitch1.27mm" H 6410 3350 50  0001 C CNN
 F 3 "" H 6510 3450 50  0000 C CNN
+F 4 "LM339DE4" H 6460 3250 60  0001 C CNN "MPN"
 	2    6460 3250
 	1    0    0    -1
@@
 F 2 "Resistors_SMD:R_0805_HandSoldering" H 4980 2620 50  0001 C CNN
 F 3 "" H 4980 2620 50  0000 C CNN
-F 4 "Value" H 4980 2620 60  0001 C CNN "Fieldname"
+F 4 "RC0805FR-072ML" H 4980 2620 60  0001 C CNN "MPN"
 	1    4980 2620
 	0    1    1    0
@@
 Connection ~ 5610 2620
 Connection ~ 4800 2620
+$Comp
+L R_Small R303
+U 1 1 5824D2B3
+P 6820 3000
+F 0 "R303" V 6900 2960 50  0000 L CNN
+F 1 "10K" V 6750 2880 50  0000 L CNN
+F 2 "Resistors_SMD:R_0805_HandSoldering" H 6820 3000 50  0001 C CNN
+F 3 "" H 6820 3000 50  0000 C CNN
+F 4 "RC0805FR-072ML" H 6820 3000 60  0001 C CNN "MPN"
+	1    6820 3000
+	-1   0    0    1
+$EndComp
+Text GLabel 6820 2750 1    60   Input ~ 0
++3V
+Wire Wire Line
+	6820 2750 6820 2900
+Wire Wire Line
+	6820 3100 6820 3250
+Connection ~ 6820 3250
 $EndSCHEMATC

Commit message: removed 10K resistors used as load for op amps
Parts:
- removed R302: 10K, Resistors_SMD:R_0805_HandSoldering, symbol R_Small
Changed lines of the file:
@@
 	5110 2100 4800 2100
-Wire Wire Line
-	5610 2100 5610 3450
 Wire Wire Line
 	5400 3150 6160 3150
@@
 	5310 2100 5610 2100
 $Comp
-L GND #PWR012
+L GND #PWR011
 U 1 1 58229142
 P 4800 3550
-F 0 "#PWR012" H 4800 3300 50  0001 C CNN
+F 0 "#PWR011" H 4800 3300 50  0001 C CNN
 F 1 "GND" H 4800 3400 50  0000 C CNN
 F 2 "" H 4800 3550 50  0000 C CNN
@@
 Wire Wire Line
 	4800 3250 4800 3550
-$Comp
-L R_Small R302
-U 1 1 5822914A
-P 5610 3550
-F 0 "R302" V 5690 3510 50  0000 L CNN
-F 1 "10K" V 5540 3430 50  0000 L CNN
-F 2 "Resistors_SMD:R_0805_HandSoldering" H 5610 3550 50  0001 C CNN
-F 3 "" H 5610 3550 50  0000 C CNN
-F 4 "Value" H 5610 3550 60  0001 C CNN "Fieldname"
-	1    5610 3550
-	-1   0    0    1
-$EndComp
-Connection ~ 5610 3150
-$Comp
-L GND #PWR013
-U 1 1 58229152
-P 5610 3750
-F 0 "#PWR013" H 5610 3500 50  0001 C CNN
-F 1 "GND" H 5610 3600 50  0000 C CNN
-F 2 "" H 5610 3750 50  0000 C CNN
-F 3 "" H 5610 3750 50  0000 C CNN
-	1    5610 3750
-	1    0    0    -1
-$EndComp
-Wire Wire Line
-	5610 3650 5610 3750
 $Comp
 L LM339 U202
@@
 	4190 3050 4800 3050
 $Comp
-L GND #PWR014
+L GND #PWR012
 U 1 1 58229194
 P 4240 3510
-F 0 "#PWR014" H 4240 3260 50  0001 C CNN
+F 0 "#PWR012" H 4240 3260 50  0001 C CNN
 F 1 "GND" H 4240 3360 50  0000 C CNN
 F 2 "" H 4240 3510 50  0000 C CNN
@@
 $EndComp
 Wire Wire Line
-	5610 2620 5080 2620
-Wire Wire Line
 	4880 2620 4800 2620
-Connection ~ 5610 2620
 Connection ~ 4800 2620
 $Comp
@@
 	6820 3100 6820 3250
 Connection ~ 6820 3250
+Wire Wire Line
+	5610 2100 5610 3150
+Connection ~ 5610 3150
+Wire Wire Line
+	5080 2620 5610 2620
+Connection ~ 5610 2620
 $EndSCHEMATC

Commit message: replaced potentiometer with trimpot
Connections:
- net GND: now also U201.2 (-); no longer U201.6 (-)
- net at C301.1, R301.1, U202.7 (+): now also U201.1; no longer U201.7
- net at C301.2, PD301.1 (K), R301.2: now also U201.3 (+); no longer U201.5 (+)
Changed lines of the file:
@@
 $Comp
 L MCP6404 U201
-U 2 1 58229131
+U 1 1 58229131
 P 5100 3150
 F 0 "U201" H 5150 3350 50  0000 C CNN
@@
 F 2 "Housings_SOIC:SOIC-14_3.9x8.7mm_Pitch1.27mm" H 5050 3250 50  0001 C CNN
 F 3 "" H 5150 3350 50  0000 C CNN
-	2    5100 3150
+	1    5100 3150
 	1    0    0    -1
 $EndComp

Commit message: completed pcb basic layout
Parts:
- renumbered R303 to R302
Changed lines of the file:
@@
 	5310 2100 5610 2100
 $Comp
-L GND #PWR011
+L GND #PWR302
 U 1 1 58229142
 P 4800 3550
-F 0 "#PWR011" H 4800 3300 50  0001 C CNN
+F 0 "#PWR302" H 4800 3300 50  0001 C CNN
 F 1 "GND" H 4800 3400 50  0000 C CNN
 F 2 "" H 4800 3550 50  0000 C CNN
@@
 	4190 3050 4800 3050
 $Comp
-L GND #PWR012
+L GND #PWR301
 U 1 1 58229194
 P 4240 3510
-F 0 "#PWR012" H 4240 3260 50  0001 C CNN
+F 0 "#PWR301" H 4240 3260 50  0001 C CNN
 F 1 "GND" H 4240 3360 50  0000 C CNN
 F 2 "" H 4240 3510 50  0000 C CNN
@@
 Connection ~ 4800 2620
 $Comp
-L R_Small R303
+L R_Small R302
 U 1 1 5824D2B3
 P 6820 3000
-F 0 "R303" V 6900 2960 50  0000 L CNN
+F 0 "R302" V 6900 2960 50  0000 L CNN
 F 1 "10K" V 6750 2880 50  0000 L CNN
 F 2 "Resistors_SMD:R_0805_HandSoldering" H 6820 3000 50  0001 C CNN

Commit message: changed photodiodes to BPW 34 S due to availability. Changed feedbak resistor and cap due to increased current output of diode.
Parts:
- C301: value 50p -> 100p; Fieldname (none) -> Value
- PD301: value VBPW34S -> BPW 34 S-Z; AltPart (none) -> VBPW34S
- R301: value 2M -> 1M; Fieldname (none) -> Value; MPN RC0805FR-072ML -> (none)
- R302: Fieldname (none) -> Value; MPN RC0805FR-072ML -> (none)
Changed lines of the file:
@@
 P 5210 2100
 F 0 "C301" V 5330 2060 50  0000 L CNN
-F 1 "50p" V 5100 1970 50  0000 L CNN
+F 1 "100p" V 5100 1970 50  0000 L CNN
 F 2 "Capacitors_SMD:C_0805_HandSoldering" H 5210 2100 50  0001 C CNN
 F 3 "" H 5210 2100 50  0000 C CNN
+F 4 "Value" H 5210 2100 60  0001 C CNN "Fieldname"
 	1    5210 2100
 	0    1    1    0
@@
 	5310 2100 5610 2100
 $Comp
-L GND #PWR302
+L GND #PWR011
 U 1 1 58229142
 P 4800 3550
-F 0 "#PWR302" H 4800 3300 50  0001 C CNN
+F 0 "#PWR011" H 4800 3300 50  0001 C CNN
 F 1 "GND" H 4800 3400 50  0000 C CNN
 F 2 "" H 4800 3550 50  0000 C CNN
@@
 P 4190 3260
 F 0 "PD301" H 4110 3340 50  0000 L CNN
-F 1 "VBPW34S" H 4040 3180 50  0000 L CNN
+F 1 "BPW 34 S-Z" H 4040 3180 50  0000 L CNN
 F 2 "DasBlinkinput:VBPW34S" V 4190 3260 50  0001 C CNN
-F 3 "http://www.vishay.com/docs/81128/vbpw34s.pdf" V 4190 3260 50  0001 C CNN
+F 3 "http://media.digikey.com/pdf/Data%20Sheets/Osram%20PDFs/bpw34_spdf.pdf" V 4190 3260 50  0001 C CNN
 F 4 "Value" H 4190 3260 60  0001 C CNN "Fieldname"
+F 5 "VBPW34S" H 4190 3260 60  0001 C CNN "AltPart"
 	1    4190 3260
 	0    1    1    0
@@
 	4190 3050 4800 3050
 $Comp
-L GND #PWR301
+L GND #PWR012
 U 1 1 58229194
 P 4240 3510
-F 0 "#PWR301" H 4240 3260 50  0001 C CNN
+F 0 "#PWR012" H 4240 3260 50  0001 C CNN
 F 1 "GND" H 4240 3360 50  0000 C CNN
 F 2 "" H 4240 3510 50  0000 C CNN
@@
 P 4980 2620
 F 0 "R301" V 5060 2580 50  0000 L CNN
-F 1 "2M" V 4910 2500 50  0000 L CNN
+F 1 "1M" V 4910 2500 50  0000 L CNN
 F 2 "Resistors_SMD:R_0805_HandSoldering" H 4980 2620 50  0001 C CNN
 F 3 "" H 4980 2620 50  0000 C CNN
-F 4 "RC0805FR-072ML" H 4980 2620 60  0001 C CNN "MPN"
+F 4 "Value" H 4980 2620 60  0001 C CNN "Fieldname"
+F 5 "  " H 4980 2620 60  0001 C CNN "MPN"
 	1    4980 2620
 	0    1    1    0
@@
 F 2 "Resistors_SMD:R_0805_HandSoldering" H 6820 3000 50  0001 C CNN
 F 3 "" H 6820 3000 50  0000 C CNN
-F 4 "RC0805FR-072ML" H 6820 3000 60  0001 C CNN "MPN"
+F 4 "Value" H 6820 3000 60  0001 C CNN "Fieldname"
 	1    6820 3000
 	-1   0    0    1

Commit message: added test points at outputs of op-amps
Parts:
- added P301: CONN_01X01, Pin_Headers:Pin_Header_Straight_1x01, symbol CONN_01X01
Connections:
- net at C301.1, R301.1, U201.1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: now also P301.1 (P1)
Changed lines of the file:
@@
 	5080 2620 5610 2620
 Connection ~ 5610 2620
+$Comp
+L CONN_01X01 P301
+U 1 1 585445D1
+P 5830 3450
+F 0 "P301" H 5780 3550 50  0000 C CNN
+F 1 "CONN_01X01" V 5930 3450 50  0000 C CNN
+F 2 "Pin_Headers:Pin_Header_Straight_1x01" H 5830 3450 50  0001 C CNN
+F 3 "" H 5830 3450 50  0000 C CNN
+	1    5830 3450
+	0    1    1    0
+$EndComp
+Wire Wire Line
+	5830 3250 5830 3150
+Connection ~ 5830 3150
 $EndSCHEMATC

Commit message: corrected inputs on opamp and rerouted traces
Parts:
- U201, U202: footprint Housings_SOIC:SOIC-14_3.9x8.7mm_Pitch1.27mm -> DasBlinkinput:SOIC-14_3.9x8.7mm_Pitch1.27mm
Connections:
- net GND: now also U201.3 (+); no longer U201.2 (-)
- net at C301.2, PD301.1 (K), R301.2: now also U201.2 (-); no longer U201.3 (+)
Changed lines of the file:
@@
 F 0 "U201" H 5150 3350 50  0000 C CNN
 F 1 "MCP6404" H 5250 2950 50  0000 C CNN
-F 2 "Housings_SOIC:SOIC-14_3.9x8.7mm_Pitch1.27mm" H 5050 3250 50  0001 C CNN
+F 2 "DasBlinkinput:SOIC-14_3.9x8.7mm_Pitch1.27mm" H 5050 3250 50  0001 C CNN
 F 3 "" H 5150 3350 50  0000 C CNN
 	1    5100 3150
-	1    0    0    -1
+	1    0    0    1
 $EndComp
 Wire Wire Line
@@
 F 0 "U202" H 6510 3450 50  0000 C CNN
 F 1 "LM339" H 6560 3050 50  0000 C CNN
-F 2 "Housings_SOIC:SOIC-14_3.9x8.7mm_Pitch1.27mm" H 6410 3350 50  0001 C CNN
+F 2 "DasBlinkinput:SOIC-14_3.9x8.7mm_Pitch1.27mm" H 6410 3350 50  0001 C CNN
 F 3 "" H 6510 3450 50  0000 C CNN
 F 4 "LM339DE4" H 6460 3250 60  0001 C CNN "MPN"
